File: _autosave-pathfinderProject.kicad_sch (KiCad schematic)
At the start: 10 parts, among them SW1 SW_Push, SW2 SW_Push, SW3 SW_Push, U1 XIAO-RP2040-DIP

Commit message: Add files via upload
Connections:
- net button1: now reaches SW1.1
- net button1: now also U1.1 (GPIO26/ADC0/A0)
- net GND: now reaches SW1.2
- net GND: now also SW2.2, SW3.2, U1.13 (GND)
- net LED2: now reaches R2.2
- net LED2: now also U1.5 (GPIO6/SDA)
- net LED3: now reaches R3.2
- net LED3: now also U1.6 (GPIO7/SCL)
- net LED1: now reaches R1.2
- net LED1: now also U1.4 (GPIO29/ADC3/A3)
- net button3: now reaches SW3.1
- net button3: now also U1.3 (GPIO28/ADC2/A2)
- net button2: now reaches U1.2 (GPIO27/ADC1/A1)
- net button2: now also SW2.1

Commit message: Add files via upload
Connections:
- net GND: now also D1.C, D2.C, D3.C
