File: pathfinderProject.kicad_sch (KiCad schematic)
At the start: 0 parts

Commit message: Add files via upload
Parts:
- added D1, D2, D3: L08R5000Q1, L08R5000Q1:LEDRD254W57D500H1070, symbol L08R5000Q1:L08R5000Q1
- added R1, R2, R3: R, symbol Device:R
- added SW1, SW2, SW3: SW_Push, symbol Switch:SW_Push
- added U1: XIAO-RP2040-DIP, Module:MOUDLE14P-XIAO-DIP-SMD, symbol Seeed_Studio_XIAO_Series:XIAO-RP2040-DIP
Connections:
- new net: D3.A, R3.1
- new net: D2.A, R2.1
- new net: D1.A, R1.1

Commit message: Add files via upload
Connections:
- net GND: now reaches D3.C
- net GND: now also D1.C, D2.C, SW1.2, SW2.2, SW3.2, U1.13 (GND)
- net button1: now reaches SW1.1
- net button1: now also U1.1 (GPIO26/ADC0/A0)
- net LED2: now reaches R2.2
- net LED2: now also U1.5 (GPIO6/SDA)
- net LED3: now reaches R3.2
- net LED3: now also U1.6 (GPIO7/SCL)
- net LED1: now reaches R1.2
- net LED1: now also U1.4 (GPIO29/ADC3/A3)
- net button3: now reaches SW3.1
- net button3: now also U1.3 (GPIO28/ADC2/A2)
- net button2: now reaches U1.2 (GPIO27/ADC1/A1)
- net button2: now also SW2.1
